Commit message: fix: update camera position

File: turtlebot3_description/urdf/turtlebot3_burger.urdf.xacro (robot description, xacro)
@@ -146,6 +146,6 @@
   <joint name="camera_joint" type="fixed">
     <axis xyz="0 1 0" />
-    <origin xyz="0.06 0 0.1" rpy="0 0.3 0"/>
-    <parent link="imu_link"/>
+    <origin xyz="0 0 1.5" rpy="0 1.2 0"/>
+    <parent link="base_link"/>
     <child link="camera_link"/>
   </joint>
